Commit message: avances

File: src/ros_sim/urdf/differential_drive.urdf (robot description, URDF)
Before this commit: robot differential_drive, 3 links, 2 joints
Links:
- added link camera_link, mass 1e-5; collision box size=0.1 0.2 0.025; visual box size=0.1 0.2 0.025
- added link imu_link, mass 1e-5; collision box size=0.1 0.1 0.025; visual box size=0.1 0.1 0.025
- link base_link: geometry collision box size=0.5 0.5 0.25; collision sphere radius=0.05
Joints:
- added joint camera_joint: type fixed, parent base_link, child camera_link, origin xyz=0.26 0 0 rpy=0 0 0, axis 0 1 0
- added joint joint_imu: type fixed, parent base_link, child imu_link, origin xyz=0 0 0.125 rpy=0 0 0
